File: m0116_usb.kicad_pcb (KiCad board)
At the start: 2 copper layers, 372.1 x 113.8 mm, 184 parts, among them J1 AVR-ISP-6, J2 USB_B_Mini, J3 Conn_01x04, J4 Conn_01x04, J5 Conn_01x06, J6 Conn_01x06, U1 ATmega32A-PU, Y1 16Mhz

Commit message: small fixes
Routing:
- net GND: track 24.6 -> 37.4 mm
- net +5V: track 431.4 -> 430.7 mm
Changed lines of the file:
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@@
     (thickness 1.6)
     (drawings 74)
-    (tracks 542)
+    (tracks 552)
     (zones 0)
     (modules 184)
@@
   (gr_line (start 88.138 89.662) (end 88.138 73.914) (layer Edge.Cuts) (width 0.05))
   (segment (start 269.5848 76.4648) (end 269.5448 76.5048) (width 0.5) (layer B.Cu) (net 1))
-  (segment (start 269.5848 73.66) (end 269.5848 76.4648) (width 0.5) (layer B.Cu) (net 1))
   (segment (start 272.0848 94.528) (end 272.0956 94.5388) (width 0.5) (layer B.Cu) (net 1))
-  (segment (start 272.0848 91.7448) (end 272.0848 94.528) (width 0.5) (layer B.Cu) (net 1))
   (segment (start 32.378 77.724) (end 31.438 78.664) (width 0.5) (layer B.Cu) (net 1))
   (segment (start 45.506 77.724) (end 32.378 77.724) (width 0.5) (layer B.Cu) (net 1))
@@
   (via (at 298.831 97.155) (size 0.8) (drill 0.4) (layers F.Cu B.Cu) (net 1))
   (via (at 297.688 82.042) (size 0.8) (drill 0.4) (layers F.Cu B.Cu) (net 1))
+  (segment (start 272.0848 94.528) (end 272.0956 94.5388) (width 0.5) (layer F.Cu) (net 1))
+  (segment (start 272.0848 91.7448) (end 272.0848 94.528) (width 0.5) (layer F.Cu) (net 1))
+  (segment (start 269.5448 73.7) (end 269.5848 73.66) (width 0.5) (layer F.Cu) (net 1))
+  (segment (start 269.5448 76.5048) (end 269.5448 73.7) (width 0.5) (layer F.Cu) (net 1))
+  (segment (start 356.108 86.36) (end 357.378 85.09) (width 0.5) (layer F.Cu) (net 1))
+  (segment (start 356.108 92.964) (end 357.505 94.361) (width 0.5) (layer F.Cu) (net 1))
+  (segment (start 379.857 82.677) (end 381.254 84.074) (width 0.5) (layer F.Cu) (net 1))
+  (segment (start 31.438 78.664) (end 31.826 78.664) (width 0.5) (layer F.Cu) (net 1))
+  (segment (start 31.826 78.664) (end 32.766 77.724) (width 0.5) (layer F.Cu) (net 1))
+  (segment (start 45.506 77.724) (end 43.815 77.724) (width 0.5) (layer F.Cu) (net 1))
+  (segment (start 75.438 92.837) (end 76.708 94.107) (width 0.5) (layer F.Cu) (net 1))
+  (segment (start 75.438 86.487) (end 76.708 85.217) (width 0.5) (layer F.Cu) (net 1))
   (segment (start 169.037 79.43) (end 175.537 79.43) (width 0.25) (layer F.Cu) (net 2))
   (segment (start 248.85299 73.59299) (end 251.7648 76.5048) (width 0.25) (layer B.Cu) (net 2))
@@
   (segment (start 236.474 89.789) (end 238.379 91.694) (width 0.25) (layer B.Cu) (net 4))
   (segment (start 236.474 86.3759) (end 236.474 89.789) (width 0.25) (layer B.Cu) (net 4))
-  (segment (start 272.0848 73.66) (end 272.0848 76.5048) (width 0.5) (layer B.Cu) (net 5))
   (segment (start 269.5448 94.488) (end 269.5956 94.5388) (width 0.5) (layer B.Cu) (net 5))
-  (segment (start 269.5448 91.7448) (end 269.5448 94.488) (width 0.5) (layer B.Cu) (net 5))
   (segment (start 269.5448 84.0232) (end 269.5448 91.7448) (width 0.5) (layer B.Cu) (net 5))
   (segment (start 272.0848 76.5048) (end 272.0848 81.4832) (width 0.5) (layer B.Cu) (net 5))
@@
   (segment (start 48.006 83.947) (end 65.278 83.947) (width 0.5) (layer F.Cu) (net 5))
   (segment (start 186.934981 96.783019) (end 195.326 88.392) (width 0.5) (layer F.Cu) (net 5))
-  (segment (start 70.414019 96.783019) (end 186.934981 96.783019) (width 0.5) (layer F.Cu) (net 5))
-  (segment (start 67.818 94.187) (end 70.414019 96.783019) (width 0.5) (layer F.Cu) (net 5))
-  (segment (start 67.818 92.837) (end 67.818 94.187) (width 0.5) (layer F.Cu) (net 5))
   (segment (start 187.814001 80.880001) (end 195.326 88.392) (width 0.5) (layer F.Cu) (net 5))
   (segment (start 162.414001 80.880001) (end 187.814001 80.880001) (width 0.5) (layer F.Cu) (net 5))
@@
   (segment (start 354.584 75.184) (end 343.408 86.36) (width 0.5) (layer B.Cu) (net 5))
   (segment (start 378.968 75.184) (end 354.584 75.184) (width 0.5) (layer B.Cu) (net 5))
+  (segment (start 269.5448 94.488) (end 269.5956 94.5388) (width 0.5) (layer F.Cu) (net 5))
+  (segment (start 269.5448 91.7448) (end 269.5448 94.488) (width 0.5) (layer F.Cu) (net 5))
+  (segment (start 272.0848 73.66) (end 272.0848 76.5048) (width 0.5) (layer F.Cu) (net 5))
+  (segment (start 67.818 92.837) (end 71.764019 96.783019) (width 0.5) (layer F.Cu) (net 5))
+  (segment (start 71.764019 96.783019) (end 186.934981 96.783019) (width 0.5) (layer F.Cu) (net 5))
   (segment (start 67.437 80.264) (end 67.818 80.645) (width 0.25) (layer F.Cu) (net 6))
   (segment (start 31.438 80.264) (end 67.437 80.264) (width 0.25) (layer F.Cu) (net 6))

Commit message: logos!
Parts:
- added G***: LOGO, custom_parts:m0116_qr, B.Cu at (305.1, 146.7)
- added G***: LOGO, custom_parts:qmk, B.Cu at (150.9, 174.2)
- added G***: LOGO, custom_parts:pear_x_elmo, B.Cu at (146.6, 91.4)
- added G***: LOGO, custom_parts:oshw, B.Cu at (137.3, 167.1)
Other:
- board text added: "M0116 USB PCB v0.1"

Commit message: gerbers
Routing:
- net (no net): track 0.00 -> 56.8 mm
- net GND: track 37.4 -> 56.4 mm
Other:
- outline, holes or cut-outs redrawn

Commit message: make JLC happy
Routing:
- net GND: track 56.4 -> 122.2 mm
- net (no net): track 56.8 -> 0.00 mm

Commit message: fix wrong resistor connection
Connections:
- R5 pad 1: Net-(J3-Pad3) -> Net-(J3-Pad2)
Routing:
- net GND: track 122.2 -> 56.4 mm
- net Net-(J3-Pad3): track 130.9 -> 116.3 mm
- net Net-(J3-Pad2): track 124.4 -> 136.7 mm
Other:
- outline, holes or cut-outs redrawn

Commit message: rev1
Parts:
- removed the C1 at (238.4, 76.2)
- removed the C2 at (238.4, 91.7)
- removed J5, J6: Conn_01x06, Connector_PinHeader_2.54mm:PinHeader_1x06_P2.54mm_Vertical
- Y1: value 16Mhz -> Resonator; footprint Crystal:Crystal_HC49-4H_Vertical -> Crystal:Resonator-3Pin_W7.0mm_H2.5mm
- moved J1 37.2 mm to (341.9, 88.9), turned to 90 degrees
- moved F1 10.4 mm to (58.4, 84.2)
- moved C1 9.14 mm to (57.1, 77.7)
- moved Boot1 8.64 mm to (169.0, 83.6)
- moved Reset1 8.25 mm to (169.0, 75.6)
- moved R1 7.33 mm to (163.3, 87.1), turned to 90 degrees
- moved C2 5.61 mm to (274.2, 97.8), turned to 90 degrees
- moved R4 5.59 mm to (190.5, 88.4)
- moved Y1 4.95 mm to (241.3, 80.4)
- moved R3 4.57 mm to (185.5, 88.4)
- moved D39 2.79 mm to (50.8, 139.8)
- moved D40 2.79 mm to (76.8, 139.8)
- moved D41 2.79 mm to (95.9, 139.8)
- moved D42 2.79 mm to (114.9, 139.8)
- moved D43 2.79 mm to (134.1, 139.8)
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- renumbered C3 to C1, C4 to C2, C5 to C3, D84 to D74, D74 to D75, D75 to D76, D76 to D77, D77 to D78, D78 to D79, D79 to D80, D80 to D81, D81 to D82, J4 to J2, MX81 to MX72, MX72 to MX73, MX73 to MX74, MX74 to MX75, MX75 to MX76, MX76 to MX77, MX77 to MX78, MX78 to MX79, MX79 to MX80, MX80 to MX81, R5 to R2, R2 to R4, J2 to USB1
Connections:
- J1 pad 1: Net-(J1-Pad1) -> MISO
- J1 pad 3: Net-(J1-Pad3) -> SCK
- J1 pad 4: Net-(J1-Pad4) -> MOSI
- J1 pad 5: Net-(J1-Pad5) -> reset
- R2 pad 1: Net-(J3-Pad2) -> Net-(J3-Pad3)
- U1 pad 12: Net-(C2-Pad1) -> Net-(U1-Pad12)
- U1 pad 16: D- -> D+
- U1 pad 17: D+ -> D-
- USB1 pad 6: Net-(J2-Pad6) -> GND
- Y1 pad 2: Net-(C2-Pad1) -> GND
Routing:
- net GND: track 56.4 -> 5.78 mm, vias 6 -> 3
- net Net-(J1-Pad4): track 46.1 -> 0.00 mm
- net +5V: track 430.7 -> 388.6 mm
- net Net-(C2-Pad1): track 40.7 -> 0.00 mm
- net Net-(J1-Pad1): track 32.5 -> 0.00 mm
- net Net-(U1-Pad12): track 0.00 -> 32.4 mm
- net Net-(J1-Pad3): track 28.9 -> 0.00 mm
- net Net-(J1-Pad5): track 25.3 -> 0.00 mm
- net Net-(J3-Pad3): track 116.3 -> 136.2 mm
- net col5: track 197.3 -> 214.7 mm
- net boot: track 86.4 -> 102.2 mm
- net MOSI: track 75.7 -> 91.1 mm
- net col6: track 206.4 -> 219.9 mm
- net Net-(J3-Pad2): track 136.7 -> 124.1 mm
- net VCC: track 12.3 -> 25.0 mm
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Other:
- outline, holes or cut-outs redrawn
- board text added: "M0116 USB PCB rev1"
- board text removed: "M0116 USB PCB v0.1"

Commit message: change design of daughterboard
Parts:
- J2: footprint Connector_PinHeader_2.54mm:PinHeader_1x04_P2.54mm_Vertical -> Connector_PinHeader_2.00mm:PinHeader_1x04_P2.00mm_Vertical
- J3: footprint Connector_PinHeader_2.54mm:PinHeader_1x04_P2.54mm_Vertical -> Connector_JST:JST_EH_B4B-EH-A_1x04_P2.50mm_Vertical
- moved J2 33.8 mm to (35.3, 77.2), turned to 0 degrees
- moved C1 28.3 mm to (85.3, 79.5), turned to 270 degrees
- moved F1 21.6 mm to (79.8, 80.8)
- moved D2 15.3 mm to (75.4, 89.4)
- moved J3 12.7 mm to (69.8, 80.3), turned to 270 degrees
- moved D1 9.23 mm to (75.4, 85.9)
Connections:
- J2 pad 2: Net-(D1-Pad1) -> Net-(J2-Pad2)
- J2 pad 3: Net-(D2-Pad1) -> Net-(J2-Pad3)
- J3 pad 1: +5V -> VCC
- J3 pad 2: Net-(J3-Pad2) -> Net-(D1-Pad1)
- J3 pad 3: Net-(J3-Pad3) -> Net-(D2-Pad1)
- R2 pad 1: Net-(J3-Pad3) -> Net-(D2-Pad1)
- R3 pad 1: Net-(J3-Pad2) -> Net-(D1-Pad1)
- R4 pad 1: Net-(J3-Pad3) -> Net-(D2-Pad1)
- USB1 pad 1: VCC -> +5V
- USB1 pad 2: Net-(D2-Pad1) -> Net-(J2-Pad3)
- USB1 pad 3: Net-(D1-Pad1) -> Net-(J2-Pad2)
Routing:
- net Net-(J3-Pad3): track 136.2 -> 0.00 mm
- net Net-(J3-Pad2): track 124.1 -> 0.00 mm
- net Net-(D2-Pad1): track 53.2 -> 143.8 mm
- net Net-(D1-Pad1): track 52.5 -> 130.4 mm
- net VCC: track 25.0 -> 5.03 mm
- net Net-(J2-Pad3): track 0.00 -> 12.3 mm
- net +5V: track 388.6 -> 394.3 mm
- net Net-(J2-Pad2): track 0.00 -> 4.30 mm
Other:
- outline, holes or cut-outs redrawn

Commit message: change JST connector size
Parts:
- removed Y1: Resonator, Crystal:Resonator-3Pin_W7.0mm_H2.5mm
- added C4: 22p, Capacitor_THT:C_Disc_D6.0mm_W2.5mm_P5.00mm, F.Cu at (241.0, 75.9)
- added C5: 22p, Capacitor_THT:C_Disc_D6.0mm_W2.5mm_P5.00mm, F.Cu at (241.0, 91.3)
- added XTAL1: Crystal, Crystal:Crystal_HC49-4H_Vertical, F.Cu at (239.0, 81.2)
- J3: footprint Connector_JST:JST_EH_B4B-EH-A_1x04_P2.50mm_Vertical -> Connector_JST:JST_PH_S4B-PH-K_1x04_P2.00mm_Horizontal
- moved J3 0.90 mm to (69.7, 81.2)
Connections:
- J2 pad 1: +5V -> VCC
- USB1 pad 1: +5V -> VCC
Routing:
- net Net-(C4-Pad1): track 26.0 -> 35.0 mm
- net Net-(C5-Pad1): track 32.4 -> 40.5 mm
- net VCC: track 5.03 -> 10.4 mm
- net +5V: track 394.3 -> 389.1 mm
- net Net-(D2-Pad1): track 143.8 -> 144.4 mm
Other:
- outline, holes or cut-outs redrawn
